File: KiCad/PreAmp/PreAmp.sch (KiCad schematic (older format))
At the start: 145 parts, among them J1 CONN_01X02, J2 CONN_01X02, J3 CONN_01X02, J4 CONN_01X02, J5 CONN_01X02, J6 CONN_01X02, K1 G6K-2F, K2 G6K-2F, K3 G6K-2F, K4 G6K-2F, K5 G6K-2F, P1 A-POWER, P13 CTRL_VOLUME, P14 RSA-IN2L, P15 RSA-IN2R, P16 RSA-IN3L, P17 RSA-IN3R, P2 RSA-IN1L, P3 RSA-INTL, P4 RSA-IN1R, P5 RSA-INTR, P8 CTRL_RELAYS, Q1 BC817, Q2 BC817, Q3 BC817, Q4 BC817, Q5 BC817, U1 78M15, U2 79M15, U3 78L05, U4 78L05, U5 79L05, U6 NE5532, U7 NE5532, U8 PGA4311, U9 TL074

Commit message: Commit
Parts:
- C1, C13, C14, C15, C2, C25, C5, C6: symbol CP -> Device:CP
- C10, C11, C12, C16, C17, C18, C19, C20, C21, C22, C26, C27, C28, C29, C3, C30, C31, C32, C33, C34, C35, C36, C37, C38, C39, C4, C7, C8, C9: symbol C -> Device:C
- D1, D10, D11, D13, D2, D5, D6, D7, D8: symbol D -> Device:D
- D12, D14, D3, D4, D9: symbol LED-RESCUE-PreAmp -> PreAmp-rescue:LED-RESCUE-PreAmp
- J1, J2, J3, J4, J5, J6: symbol CONN_01X02 -> PreAmp-rescue:CONN_01X02
- K1, K2, K3, K4, K5: symbol G6K-2F -> PreAmp-rescue:G6K-2F
- P1: symbol CONN_01X04 -> PreAmp-rescue:CONN_01X04
- P13: symbol CONN_02X04 -> PreAmp-rescue:CONN_02X04
- P14, P15, P16, P17, P2, P3, P4, P5: symbol BNC -> PreAmp-rescue:BNC
- P8: symbol CONN_01X10 -> PreAmp-rescue:CONN_01X10
- Q1, Q2, Q3, Q4, Q5: symbol Q_NPN_BEC -> Device:Q_NPN_BEC
- R1, R10, R11, R12, R13, R14, R15, R16, R17, R18, R19, R2, R20, R21, R22, R23, R24, R25, R26, R27, R28, R29, R3, R30, R31, R32, R33, R34, R35, R36, R37, R38, R39, R4, R40, R41, R42, R43, R44, R45, R46, R47, R48, R49, R5, R50, R51, R52, R53, R54, R55, R56, R57, R58, R6, R7, R8, R9: symbol R -> Device:R
- U1: symbol LM7815CT -> PreAmp-rescue:LM7815CT
- U2: symbol LM7915CT -> PreAmp-rescue:LM7915CT
- U3, U4: symbol LM78L05ACZ -> PreAmp-rescue:LM78L05ACZ
- U5: symbol LM7905CT -> PreAmp-rescue:LM7905CT
- U6, U7: symbol NE5532 -> PreAmp-rescue:NE5532
- U8: symbol PGA4311 -> PreAmp-rescue:PGA4311
- U9: symbol TL074-RESCUE-PreAmp -> PreAmp-rescue:TL074-RESCUE-PreAmp
