File: KiCad/PreAmp/PreAmp.sch (KiCad schematic (older format))
At the start: 144 parts, among them J1 CONN_01X02, J2 CONN_01X02, J3 CONN_01X02, J4 CONN_01X02, J5 CONN_01X02, J6 CONN_01X02, K1 G6K-2F, K2 G6K-2F, K3 G6K-2F, K4 G6K-2F, K5 G6K-2F, P1 A-POWER, P13 CTRL_VOLUME, P14 RSA-IN2L, P15 RSA-IN2R, P16 RSA-IN3L, P17 RSA-IN3R, P2 RSA-IN1L, P3 RSA-INTL, P4 RSA-IN1R, P5 RSA-INTR, P8 CTRL_RELAYS, Q1 BC817, Q2 BC817, Q3 BC817, Q4 BC817, Q5 BC817, U1 78M15, U2 79M15, U3 78L05, U4 78L05, U5 79L05, U6 NE5532, U7 NE5532, U8 PGA4311, U9 TL074

Commit message: Last tweaks
Parts:
- added R58: 0, Resistor_SMD:R_0805_2012Metric, symbol Device:R
- C13: footprint Capacitor_THT:CP_Radial_D6.3mm_P2.50mm -> Capacitor_SMD:C_Elec_6.3x5.8
Connections:
- net GNDA: now also R58.2
- net GNDPWR: now also R58.1
Changed lines of the file:
@@
 F 0 "C13" H 14525 6350 50  0000 L CNN
 F 1 "47u" H 14525 6150 50  0000 L CNN
-F 2 "Capacitor_THT:CP_Radial_D6.3mm_P2.50mm" H 14538 6100 50  0001 C CNN
+F 2 "Capacitor_SMD:C_Elec_6.3x5.8" H 14538 6100 50  0001 C CNN
 F 3 "" H 14500 6250 50  0000 C CNN
 	1    14500 6250
@@
 Wire Wire Line
 	10950 7100 10850 7100
+$Comp
+L power:GNDPWR #PWR0123
+U 1 1 5DF852EC
+P 12650 5700
+F 0 "#PWR0123" H 12650 5500 50  0001 C CNN
+F 1 "GNDPWR" V 12655 5592 50  0000 R CNN
+F 2 "" H 12650 5650 50  0001 C CNN
+F 3 "" H 12650 5650 50  0001 C CNN
+	1    12650 5700
+	0    -1   -1   0
+$EndComp
+$Comp
+L power:GNDA #PWR0124
+U 1 1 5DF85435
+P 12350 5700
+F 0 "#PWR0124" H 12350 5450 50  0001 C CNN
+F 1 "GNDA" H 12350 5550 50  0000 C CNN
+F 2 "" H 12350 5700 50  0000 C CNN
+F 3 "" H 12350 5700 50  0000 C CNN
+	1    12350 5700
+	0    1    1    0
+$EndComp
+$Comp
+L Device:R R58
+U 1 1 5DF85A76
+P 12500 5700
+F 0 "R58" V 12580 5700 50  0000 C CNN
+F 1 "0" V 12500 5700 50  0000 C CNN
+F 2 "Resistor_SMD:R_0805_2012Metric" V 12430 5700 50  0001 C CNN
+F 3 "" H 12500 5700 50  0000 C CNN
+	1    12500 5700
+	0    1    1    0
+$EndComp
 $EndSCHEMATC

Commit message: Silk stuff
Connections:
- net GNDA: now also J2.2 (P2), J3.2 (P2); no longer J2.1 (P1), J3.1 (P1)
- net OUT-TB-L: now also J2.1 (P1); no longer J2.2 (P2)
- net OUT-TB-R: now also J3.1 (P1); no longer J3.2 (P2)
Changed lines of the file:
@@
 F 3 "" H 9350 3450 50  0001 C CNN
 	1    9350 3450
-	1    0    0    1
+	1    0    0    -1
 $EndComp
 $Comp
@@
 F 3 "" H 9350 4500 50  0001 C CNN
 	1    9350 4500
-	1    0    0    1
+	1    0    0    -1
 $EndComp
 Wire Wire Line
