File: KiCad/PreAmp/_saved_PreAmp.sch (KiCad schematic (older format))
At the start: 144 parts, among them J1 CONN_01X02, J2 CONN_01X02, J3 CONN_01X02, J4 CONN_01X02, J5 CONN_01X02, J6 CONN_01X02, K1 G6K-2F, K2 G6K-2F, K3 G6K-2F, K4 G6K-2F, K5 G6K-2F, P1 A-POWER, P13 CTRL_VOLUME, P14 RSA-IN2L, P15 RSA-IN2R, P16 RSA-IN3L, P17 RSA-IN3R, P2 RSA-IN1L, P3 RSA-INTL, P4 RSA-IN1R, P5 RSA-INTR, P8 CTRL_RELAYS, Q1 BC817, Q2 BC817, Q3 BC817, Q4 BC817, Q5 BC817, U1 78M15, U2 79M15, U3 78L05, U4 78L05, U5 79L05, U6 NE5532, U7 NE5532, U8 PGA4311, U9 TL074

Commit message: PreAmp PCP pimped
Parts:
- C13: footprint Capacitor_THT:CP_Radial_D6.3mm_P2.50mm -> Capacitor_SMD:C_Elec_6.3x5.8
Changed lines of the file:
@@
 F 0 "C13" H 14525 6350 50  0000 L CNN
 F 1 "47u" H 14525 6150 50  0000 L CNN
-F 2 "Capacitor_THT:CP_Radial_D6.3mm_P2.50mm" H 14538 6100 50  0001 C CNN
+F 2 "Capacitor_SMD:C_Elec_6.3x5.8" H 14538 6100 50  0001 C CNN
 F 3 "" H 14500 6250 50  0000 C CNN
 	1    14500 6250
