File: KiCad/PowerAmp/PowerAmp.kicad_pcb (KiCad board)
At the start: 2 copper layers, 95.9 x 45.1 mm, 47 parts, among them P1 OUT-L, P2 IN-L, P3 POWER, P4 MUTE, P5 OUT-R, P6 IN-R, Q1 BC846, Q2 BC846, Q3 BC856, Q4 BC846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

Commit message: Power Amp board v3
Parts:
- added C12: 220n, Capacitor_SMD:C_0805_2012Metric, B.Cu at (103.5, 68.6)
- added C13: 220n, Capacitor_SMD:C_0805_2012Metric, B.Cu at (100.3, 68.6)
- added C17: 1u, Capacitor_SMD:C_2220_5650Metric, F.Cu at (68.6, 66.0)
- added C18: 1u, Capacitor_SMD:C_2220_5650Metric, F.Cu at (118.1, 66.0)
- added L1: L, Inductor_THT:L_Axial_L9.5mm_D4.0mm_P12.70mm_Horizontal_Fastron_SMCC, F.Cu at (50.2, 78.7)
- added L2: L, Inductor_THT:L_Axial_L9.5mm_D4.0mm_P12.70mm_Horizontal_Fastron_SMCC, F.Cu at (96.5, 78.7)
- added R16: 47, Resistor_SMD:R_0805_2012Metric, B.Cu at (81.3, 54.0)
- C1, C7: footprint Capacitors_SMD:C_0805 -> Capacitor_SMD:C_0805_2012Metric
- C10, C11: footprint Capacitors_THT:CP_Radial_D5.0mm_P2.50mm -> Capacitor_THT:CP_Radial_D5.0mm_P2.00mm
- C14: value 22u -> 22u/63V; footprint Capacitors_THT:CP_Radial_D5.0mm_P2.50mm -> Capacitor_THT:CP_Radial_D5.0mm_P2.50mm
- C15, C5: footprint Capacitors_THT:CP_Radial_D5.0mm_P2.50mm -> Capacitor_Tantalum_SMD:CP_EIA-6032-28_Kemet-C; moved to B.Cu
- C16, C6: value 470n -> 1u; footprint Capacitors_SMD:C_0805 -> Capacitor_SMD:C_2220_5650Metric; moved to F.Cu
- C2, C3, C8, C9: footprint Capacitors_THT:CP_Radial_D18.0mm_P7.50mm -> Capacitor_THT:CP_Radial_D18.0mm_P7.50mm
- C4: value 22u -> 22u/63V; footprint Capacitors_THT:CP_Radial_D5.0mm_P2.50mm -> Capacitor_THT:CP_Radial_D5.0mm_P2.00mm
- D1: footprint Diodes_SMD:D_1206 -> Diode_SMD:D_MiniMELF
- P2, P4, P6: footprint Connect:PINHEAD1-2 -> Connector_Molex:Molex_Micro-Latch_53253-0270_1x02_P2.00mm_Vertical
- P3: footprint Connectors_Molex:Molex_MiniFit-JR-5556-04A_2x02x4.20mm_Straight -> Connector_Molex:Molex_Mini-Fit_Jr_5566-04A_2x02_P4.20mm_Vertical
- Q1, Q2, Q3, Q4: footprint TO_SOT_Packages_SMD:SOT-23 -> Package_TO_SOT_SMD:SOT-23
- R1, R10, R11, R12, R13, R14, R15, R2, R3, R4, R5, R6, R7, R8, R9: footprint Resistors_SMD:R_0805 -> Resistor_SMD:R_0805_2012Metric
- moved C2 50.6 mm to (71.8, 44.5)
- moved C9 50.6 mm to (101.6, 52.1)
- moved C1 41.2 mm to (57.1, 68.6), turned to 180 degrees
- moved C7 32.6 mm to (54.0, 68.6), turned to 180 degrees
- moved P5 29.1 mm to (96.5, 61.6)
- moved C3 17.9 mm to (120.0, 47.6)
- moved C8 17.9 mm to (53.3, 55.2)
- moved C16 15.3 mm to (123.8, 66.0), turned to 90 degrees
- moved R4 13.9 mm to (84.5, 57.8), turned to 270 degrees
- moved R5 10.9 mm to (86.4, 57.1), turned to 90 degrees
- moved Q1 10.3 mm to (88.9, 57.1), turned to 0 degrees
- moved C6 7.85 mm to (74.3, 66.0), turned to 90 degrees
- moved Q2 7.37 mm to (88.6, 64.9), turned to 180 degrees
- moved R10 6.75 mm to (116.8, 69.2), turned to 0 degrees
- moved R1 6.54 mm to (74.9, 78.1), turned to 90 degrees
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Connections:
- C10 pad 2: GND -> GNDA
- C11 pad 2: GND -> GNDA
- C15 pad 2: GND -> GNDA
- C5 pad 2: GND -> GNDA
- P1 pad 1: /OutL -> Net-(L1-Pad2)
- P2 pad 1: GND -> GNDA
- P4 pad 1: GND -> GNDA
- P5 pad 1: /OutR -> Net-(L2-Pad2)
- P6 pad 1: GND -> GNDA
- Q1 pad 2: GND -> GNDA
- Q2 pad 2: GND -> GNDA
- Q4 pad 2: GND -> GNDA
- R10 pad 2: GND -> GNDA
- R13 pad 2: GND -> GNDA
- R3 pad 2: GND -> GNDA
- R5 pad 2: GND -> GNDA
- U1 pad 1: GND -> GNDA
- U1 pad 4: GND -> GNDA
- U2 pad 1: GND -> GNDA
- U2 pad 4: GND -> GNDA
Routing:
- net GNDA: track 0.00 -> 123.9 mm, vias 0 -> 1
- net GND: track 202.3 -> 123.2 mm, vias 2 -> 0
- net VDD: track 158.1 -> 196.3 mm, vias 2 -> 6
- net /OutL: track 45.7 -> 32.5 mm
- net Net-(Q1-Pad3): track 4.44 -> 14.3 mm
- net /InR: track 3.92 -> 11.5 mm
- net VSS: track 145.7 -> 138.2 mm, vias 1 -> 6
- net /InL: track 4.56 -> 11.5 mm
- net Net-(C17-Pad1): track 6.52 -> 13.4 mm
- net /OutR: track 36.8 -> 30.8 mm
- net Net-(L1-Pad2): track 0.00 -> 5.98 mm
- net Net-(R1-Pad2): track 10.3 -> 5.87 mm
- net Net-(C16-Pad1): track 10.4 -> 13.9 mm
- net Net-(D1-Pad1): track 13.4 -> 9.96 mm
- net Net-(R8-Pad2): track 9.26 -> 5.87 mm
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- removed copper zone on B.Cu, net GND
- removed copper zone on F.Cu, net GND
Other:
- net class Controll added: clearance 0.2, trace_width 0.762, via_dia 2, via_drill 0.8
- board text added: "Gnd"
- board text added: "In"
- board text added: "Mute"
- board text added: "PowerAmp v3 JP, 27.07.2019"
- board text removed: "PowerAmp v2 JP, 5.09.2017"

Commit message: Small tweaks
Parts:
- P1, P5: footprint Connect:PINHEAD1-2 -> Connector_Molex:Molex_Mini-Fit_Jr_5566-02A_2x01_P4.20mm_Vertical
- moved P1 5.77 mm to (43.7, 69.8), turned to 180 degrees
- moved P5 4.02 mm to (95.2, 65.4), turned to 180 degrees
- moved C13 3.17 mm to (102.2, 66.0)
- moved L2 2.54 mm to (96.5, 81.3)
- moved C7 2.29 mm to (55.2, 66.7)
- moved C8 1.80 mm to (52.1, 56.5)
- moved C3 1.80 mm to (121.3, 48.9)
- moved P6 1.27 mm to (111.1, 65.4)
- moved C12 0.64 mm to (103.5, 67.9)
- moved C1 0.63 mm to (56.5, 68.6)
- moved L1 0.63 mm to (49.5, 78.7)
Routing:
- net VDD: track 196.3 -> 204.1 mm
- net VSS: track 138.2 -> 143.0 mm
- net GND: track 123.2 -> 125.4 mm
- net GNDA: track 123.9 -> 126.0 mm
- net Net-(L1-Pad2): track 5.98 -> 7.42 mm
- net /InR: track 11.5 -> 12.7 mm
- net /OutR: track 30.8 -> 31.6 mm
- net xMute: track 64.2 -> 63.4 mm
- net /OutL: track 32.5 -> 31.9 mm
- net Net-(L2-Pad2): track 3.18 -> 3.70 mm
Other:
- board text added: "PowerAmp v3 JP, 30.07.2019"
- board text removed: "PowerAmp v3 JP, 27.07.2019"
