File: KiCad/PowerAmp/PowerAmp.sch (KiCad schematic (older format))
At the start: 42 parts, among them P1 OUT-L, P2 IN-L, P3 POWER, P4 MUTE, P5 OUT-R, P6 IN-R, Q1 BC846, Q2 BC846, Q3 BC856, Q4 BC846, U1 TDA7294V, U2 TDA7294V

Commit message: Fixes in controller app
Parts:
- C1, C16, C6, C7: symbol C -> Device:C
- C10, C11, C14, C15, C2, C3, C4, C5, C8, C9: symbol CP -> Device:CP
- D1: symbol D -> Device:D
- P1, P2, P4, P5, P6: symbol CONN_01X02 -> PowerAmp-rescue:CONN_01X02
- P3: symbol CONN_01X04 -> PowerAmp-rescue:CONN_01X04
- Q1, Q2, Q4: symbol Q_NPN_BEC -> Device:Q_NPN_BEC
- Q3: symbol Q_PNP_BEC -> Device:Q_PNP_BEC
- R1, R10, R11, R12, R13, R14, R15, R2, R3, R4, R5, R6, R7, R8, R9: symbol R -> Device:R
- U1, U2: symbol TDA7294V -> PowerAmp-rescue:TDA7294V

Commit message: Power Amp board v3
Parts:
- added C12, C13: 220n, Capacitor_SMD:C_0805_2012Metric, symbol Device:C
- added C17, C18: 1u, Capacitor_SMD:C_2220_5650Metric, symbol Device:C
- added L1, L2: L, Inductor_THT:L_Axial_L9.5mm_D4.0mm_P12.70mm_Horizontal_Fastron_SMCC, symbol Device:L
- added R16: 47, Resistor_SMD:R_0805_2012Metric, symbol Device:R
- C1, C7: footprint Capacitors_SMD:C_0805 -> Capacitor_SMD:C_0805_2012Metric
- C10, C11: footprint Capacitors_THT:CP_Radial_D5.0mm_P2.50mm -> Capacitor_THT:CP_Radial_D5.0mm_P2.00mm
- C14: value 22u -> 22u/63V; footprint Capacitors_THT:CP_Radial_D5.0mm_P2.50mm -> Capacitor_THT:CP_Radial_D5.0mm_P2.50mm
- C15, C5: footprint Capacitors_THT:CP_Radial_D5.0mm_P2.50mm -> Capacitor_Tantalum_SMD:CP_EIA-6032-28_Kemet-C
- C16, C6: value 470n -> 1u; footprint Capacitors_SMD:C_0805 -> Capacitor_SMD:C_2220_5650Metric
- C2, C3, C8, C9: footprint Capacitors_THT:CP_Radial_D18.0mm_P7.50mm -> Capacitor_THT:CP_Radial_D18.0mm_P7.50mm
- C4: value 22u -> 22u/63V; footprint Capacitors_THT:CP_Radial_D5.0mm_P2.50mm -> Capacitor_THT:CP_Radial_D5.0mm_P2.00mm
- D1: footprint Diodes_SMD:D_1206 -> Diode_SMD:D_MiniMELF
- P2, P4, P6: footprint Connect:PINHEAD1-2 -> Connector_Molex:Molex_Micro-Latch_53253-0270_1x02_P2.00mm_Vertical
- P3: footprint Connectors_Molex:Molex_MiniFit-JR-5556-04A_2x02x4.20mm_Straight -> Connector_Molex:Molex_Mini-Fit_Jr_5566-04A_2x02_P4.20mm_Vertical
- Q1, Q2, Q3, Q4: footprint TO_SOT_Packages_SMD:SOT-23 -> Package_TO_SOT_SMD:SOT-23
- R1, R10, R11, R12, R13, R14, R15, R2, R3, R4, R5, R6, R7, R8, R9: footprint Resistors_SMD:R_0805 -> Resistor_SMD:R_0805_2012Metric
Connections:
- net GND: now also C12.2, C13.1, R16.1; no longer C10.2, C11.2, C15.2, C5.2, P2.1 (P1), P4.1 (P1), P6.1 (P1), Q1.2 (E), Q2.2 (E), Q4.2 (E), R10.2, R13.2, R3.2, R5.2, U1.1 (STBY-GND), U1.4 (IN+MUTE), U2.1 (STBY-GND), U2.4 (IN+MUTE)
- net InL: now also C17.2
- net InR: now also C18.2
- net OutL: now also L1.1; no longer P1.1 (P1)
- net OutR: now also L2.1; no longer P5.1 (P1)
- net VDD: now also C12.1
- net VSS: now also C13.2
- net at C6.1, R3.1, U1.3 (IN+): now also C17.1
- net at C16.1, R10.1, U2.3 (IN+): now also C18.1
- new net: L1.2, P1.1 (P1)
- new net: L2.2, P5.1 (P1)
- new net GNDA: C10.2, C11.2, C15.2, C5.2, P2.1 (P1), P4.1 (P1), P6.1 (P1), Q1.2 (E), Q2.2 (E), Q4.2 (E), R10.2, R13.2, R16.2, R3.2, R5.2, U1.1 (STBY-GND), U1.4 (IN+MUTE), U2.1 (STBY-GND), U2.4 (IN+MUTE)
Other:
- moved on the sheet: C3, C7, C8, C9, P1, P2, P5, P6, R10, R3

Commit message: Small tweaks
Parts:
- C15, C5: value 22u -> 22u/25V
- P1, P5: footprint Connect:PINHEAD1-2 -> Connector_Molex:Molex_Mini-Fit_Jr_5566-02A_2x01_P4.20mm_Vertical
Changed lines of the file:
@@
 P 6050 1600
 F 0 "C5" H 6075 1700 50  0000 L CNN
-F 1 "22u" H 6075 1500 50  0000 L CNN
+F 1 "22u/25V" H 6075 1500 50  0000 L CNN
 F 2 "Capacitor_Tantalum_SMD:CP_EIA-6032-28_Kemet-C" H 6088 1450 50  0001 C CNN
 F 3 "" H 6050 1600 50  0000 C CNN
@@
 F 0 "P1" H 8850 2000 50  0000 C CNN
 F 1 "OUT-L" V 8950 1850 50  0000 C CNN
-F 2 "Connect:PINHEAD1-2" H 8850 1850 50  0001 C CNN
+F 2 "Connector_Molex:Molex_Mini-Fit_Jr_5566-02A_2x01_P4.20mm_Vertical" H 8850 1850 50  0001 C CNN
 F 3 "" H 8850 1850 50  0000 C CNN
 	1    8850 1850
@@
 P 6050 3650
 F 0 "C15" H 6075 3750 50  0000 L CNN
-F 1 "22u" H 6075 3550 50  0000 L CNN
+F 1 "22u/25V" H 6075 3550 50  0000 L CNN
 F 2 "Capacitor_Tantalum_SMD:CP_EIA-6032-28_Kemet-C" H 6088 3500 50  0001 C CNN
 F 3 "" H 6050 3650 50  0000 C CNN
@@
 F 0 "P5" H 8850 4050 50  0000 C CNN
 F 1 "OUT-R" V 8950 3900 50  0000 C CNN
-F 2 "Connect:PINHEAD1-2" H 8850 3900 50  0001 C CNN
+F 2 "Connector_Molex:Molex_Mini-Fit_Jr_5566-02A_2x01_P4.20mm_Vertical" H 8850 3900 50  0001 C CNN
 F 3 "" H 8850 3900 50  0000 C CNN
 	1    8850 3900
