File: KiCad/PowerSupply/PowerSupply.kicad_pcb (KiCad board)
At the start: 2 copper layers, 83.8 x 127 mm, 41 parts, among them P1 POWER_IN, P2 OUT, P3 OUT, P4 OUT, P5 I2C, U1 INA169, U2 MCP3426, U4 MC78L18, U5 MC78L05

Commit message: Small tweaks
Parts:
- R2: value 1k -> 10k?
- R7, R8: value 1k -> 10k
Changed lines of the file:
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@@
-(kicad_pcb (version 4) (host pcbnew 4.0.6)
+(kicad_pcb (version 20171130) (host pcbnew "(5.0.2)-1")
   (general
-    (links 89)
-    (no_connects 0)
-    (area 12.032857 24.035 104.807143 151.57)
     (thickness 1.6)
     (drawings 5)
@@
   )
   (setup
-    (last_trace_width 0.635)
+    (last_trace_width 0.25)
     (user_trace_width 0.635)
     (trace_clearance 0.2)
@@
     (pad_drill 3.2)
     (pad_to_mask_clearance 0)
+    (solder_mask_min_width 0.25)
     (aux_axis_origin 0 0)
     (visible_elements 7FFFFF9F)
@@
       (layerselection 0x00030_80000001)
       (usegerberextensions false)
+      (usegerberattributes false)
+      (usegerberadvancedattributes false)
+      (creategerberjobfile false)
       (excludeedgelayer true)
       (linewidth 0.100000)
@@
       (hpglpennumber 1)
       (hpglpenspeed 20)
-      (hpglpendiameter 15)
-      (hpglpenoverlay 2)
+      (hpglpendiameter 15.000000)
       (psnegative false)
       (psa4output false)
@@
       (net 7 GND))
     (model Capacitors_ThroughHole.3dshapes/C_Radial_D35_L51_P10.wrl
-      (at (xyz 0.19685 0 0))
+      (offset (xyz 4.999989924907684 0 0))
       (scale (xyz 1 1 1))
       (rotate (xyz 0 0 90))
@@
       (net 7 GND))
     (model Capacitors_ThroughHole.3dshapes/C_Radial_D5_L6_P2.5.wrl
-      (at (xyz 0.0492126 0 0))
+      (offset (xyz 1.250000021226883 0 0))
       (scale (xyz 1 1 1))
       (rotate (xyz 0 0 90))
@@
       (net 15 "Net-(D5-Pad2)"))
     (model LEDs.3dshapes/LED-5MM.wrl
-      (at (xyz 0.05 0 0))
+      (offset (xyz 1.269999980926514 0 0))
       (scale (xyz 1 1 1))
       (rotate (xyz 0 0 90))
@@
       (net 7 GND))
     (model LEDs.3dshapes/LED-5MM.wrl
-      (at (xyz 0.05 0 0))
+      (offset (xyz 1.269999980926514 0 0))
       (scale (xyz 1 1 1))
       (rotate (xyz 0 0 90))
@@
       (net 3 "Net-(C2-Pad2)"))
     (model Capacitors_ThroughHole.3dshapes/C_Radial_D35_L51_P10.wrl
-      (at (xyz 0.19685 0 0))
+      (offset (xyz 4.999989924907684 0 0))
       (scale (xyz 1 1 1))
       (rotate (xyz 0 0 90))
@@
       (net 7 GND))
     (model Capacitors_ThroughHole.3dshapes/C_Radial_D35_L51_P10.wrl
-      (at (xyz 0.19685 0 0))
+      (offset (xyz 4.999989924907684 0 0))
       (scale (xyz 1 1 1))
       (rotate (xyz 0 0 90))
@@
       (net 3 "Net-(C2-Pad2)"))
     (model Capacitors_ThroughHole.3dshapes/C_Radial_D35_L51_P10.wrl
-      (at (xyz 0.19685 0 0))
+      (offset (xyz 4.999989924907684 0 0))
       (scale (xyz 1 1 1))
       (rotate (xyz 0 0 90))
@@
       (net 11 +3V3))
     (model Pin_Headers.3dshapes/Pin_Header_Straight_1x04_Pitch2.54mm.wrl
-      (at (xyz 0 -0.15 0))
+      (offset (xyz 0 -3.809999942779541 0))
       (scale (xyz 1 1 1))
       (rotate (xyz 0 0 90))
@@
       (effects (font (size 1 1) (thickness 0.15)) (justify mirror))
     )
-    (fp_text value 1k (at 0 -1.75) (layer B.Fab)
+    (fp_text value 10k? (at 0 -1.75) (layer B.Fab)
       (effects (font (size 1 1) (thickness 0.15)) (justify mirror))
     )
@@
       (effects (font (size 1 1) (thickness 0.15)) (justify mirror))
     )
-    (fp_text value 1k (at 0 -1.75) (layer B.Fab)
+    (fp_text value 10k (at 0 -1.75) (layer B.Fab)
       (effects (font (size 1 1) (thickness 0.15)) (justify mirror))
     )
@@
       (effects (font (size 1 1) (thickness 0.15)) (justify mirror))
     )
-    (fp_text value 1k (at 0 -1.75) (layer B.Fab)
+    (fp_text value 10k (at 0 -1.75) (layer B.Fab)
       (effects (font (size 1 1) (thickness 0.15)) (justify mirror))
     )
@@
       (net 7 GND))
     (model ${KISYS3DMOD}/TO_SOT_Packages_SMD.3dshapes/SOT89-3_Housing.wrl
-      (at (xyz 0.02 0 0))
+      (offset (xyz 0.5079999923706054 0 0))
       (scale (xyz 0.39 0.39 0.39))
       (rotate (xyz 0 0 90))
@@
       (net 7 GND))
     (model ${KISYS3DMOD}/TO_SOT_Packages_SMD.3dshapes/SOT89-3_Housing.wrl
-      (at (xyz 0.02 0 0))
+      (offset (xyz 0.5079999923706054 0 0))
       (scale (xyz 0.39 0.39 0.39))
       (rotate (xyz 0 0 90))
