File: KiCad/PowerSupply/PowerSupply.sch (KiCad schematic (older format))
At the start: 37 parts, among them P1 POWER_IN, P2 OUT, P3 OUT, P4 OUT, P5 I2C, U1 INA169, U2 MCP3426, U4 MC78L18, U5 MC78L05

Commit message: Last tweaks
Parts:
- C1, C10, C11, C13, C14, C15, C2, C3, C4, C9: symbol C -> Device:C
- C12, C5, C6, C7, C8: symbol CP -> Device:CP
- D1: symbol Diode_Bridge-RESCUE-PowerSupply -> PowerSupply-rescue:Diode_Bridge-RESCUE-PowerSupply
- D5, D6: symbol LED-RESCUE-PowerSupply -> PowerSupply-rescue:LED-RESCUE-PowerSupply
- F1, F2: symbol FUSE -> PowerSupply-rescue:FUSE
- P1, P2, P3, P4, P5: symbol CONN_01X04 -> PowerSupply-rescue:CONN_01X04
- R1, R2, R3, R4, R5, R6, R7, R8: symbol R -> Device:R
- U1: symbol INA169 -> myLib:INA169
- U2: symbol MCP3426 -> myLib:MCP3426
- U4: symbol MC78L05ACH -> PowerSupply-rescue:MC78L05ACH
- U5: symbol MC78L18ACP -> PowerSupply-rescue:MC78L18ACP

Commit message: Small tweaks
Parts:
- C10: value ? -> 4u7
- R7, R8: value 20k -> 10k
Changed lines of the file:
@@
 P 5850 2350
 F 0 "C10" H 5875 2450 50  0000 L CNN
-F 1 "?" H 5875 2250 50  0000 L CNN
+F 1 "4u7" H 5875 2250 50  0000 L CNN
 F 2 "Capacitors_SMD:C_0805" H 5888 2200 50  0001 C CNN
 F 3 "" H 5850 2350 50  0000 C CNN
@@
 P 4600 3250
 F 0 "R7" V 4680 3250 50  0000 C CNN
-F 1 "20k" V 4600 3250 50  0000 C CNN
+F 1 "10k" V 4600 3250 50  0000 C CNN
 F 2 "Resistors_SMD:R_0805" V 4530 3250 50  0001 C CNN
 F 3 "" H 4600 3250 50  0000 C CNN
@@
 P 4850 3850
 F 0 "R8" V 4930 3850 50  0000 C CNN
-F 1 "20k" V 4850 3850 50  0000 C CNN
+F 1 "10k" V 4850 3850 50  0000 C CNN
 F 2 "Resistors_SMD:R_0805" V 4780 3850 50  0001 C CNN
 F 3 "" H 4850 3850 50  0000 C CNN
